Commit message: infrastructure changes for namespaces

File: src/zed-ros-wrapper/zed_wrapper/urdf/zed.urdf (robot description, URDF)
Before this commit: robot zed_camera, 6 links, 5 joints
Links:
- removed link base_link_c
- added link racecar2/base_link_c
Joints:
- joint zed_camera_center_joint: parent base_link_c -> racecar2/base_link_c

Commit message: Architechture changes

File: src/zed-ros-wrapper/zed_wrapper/urdf/zed.urdf (robot description, URDF)
Before this commit: robot zed_camera, 6 links, 5 joints
Links:
- removed link zed_camera_center
- removed link zed_left_camera_frame
- removed link zed_left_camera_optical_frame
- removed link zed_right_camera_frame
- removed link zed_right_camera_optical_frame
- added link racecar2/zed_camera_center; visual mesh filename=package://zed_wrapper/urdf/models/ZED.stl
- added link racecar2/zed_left_camera_frame
- added link racecar2/zed_left_camera_optical_frame
- added link racecar2/zed_right_camera_frame
- added link racecar2/zed_right_camera_optical_frame
Joints:
- removed joint zed_camera_center_joint
- removed joint zed_left_camera_joint
- removed joint zed_left_camera_optical_joint
- removed joint zed_right_camera_joint
- removed joint zed_right_camera_optical_joint
- added joint racecar2/zed_camera_center_joint: type fixed, parent racecar2/base_link_c, child racecar2/zed_camera_center, origin xyz=0 0 0 rpy=0 0 0
- added joint racecar2/zed_left_camera_joint: type fixed, parent racecar2/zed_camera_center, child racecar2/zed_left_camera_frame, origin xyz=0 0.06 0 rpy=0 0 0
- added joint racecar2/zed_left_camera_optical_joint: type fixed, parent racecar2/zed_left_camera_frame, child racecar2/zed_left_camera_optical_frame, origin xyz=0 0 0 rpy=-1.57079632679 0.0 -1.57079632679
- added joint racecar2/zed_right_camera_joint: type fixed, parent racecar2/zed_camera_center, child racecar2/zed_right_camera_frame, origin xyz=0 -0.06 0 rpy=0 0 0
- added joint racecar2/zed_right_camera_optical_joint: type fixed, parent racecar2/zed_right_camera_frame, child racecar2/zed_right_camera_optical_frame, origin xyz=0 0 0 rpy=-1.57079632679 0.0 -1.57079632679
